Commit message: FSF-4929 | launch files + fixed control (#365)
added launch files for more disciplines in pacsim
fixed error in control node due to acos not clamped to [-1, 1], resulting in NaN steering
fixed car model not appearing in foxglove

File: src/pacsim/urdf/separate_model.xacro (robot description, xacro)
@@ -1,17 +1,17 @@
 <robot name="RosE" xmlns:xacro="http://www.ros.org/wiki/xacro">
   <xacro:property name="baseFrame" value="car" />
-  <link name="${baseFrame}">
+  <link name="car">
     <visual>
       <origin rpy="0.0 0 0" xyz="0 0 0"/>
-        <geometry>
+      <geometry>
         <cylinder radius="0.001" length=".001" />
       </geometry>
     </visual>
   </link>
-   <link name="Modell">
+  <link name="Modell">
     <visual>
       <origin xyz="0 0 0" rpy="-1.57 0 0" />
       <geometry>
-      <mesh filename="package://pacsim/urdf/Model_without_Steering_Tires.stl" scale="0.01 0.01 0.01"/>
+        <mesh filename="package://pacsim/urdf/Model_without_Steering_Tires.stl" scale="0.01 0.01 0.01"/>
       </geometry>
     </visual>
@@ -21,7 +21,7 @@
       <origin rpy="-1.57 0 0" xyz="0 0 0"/>
       <geometry>
-      <mesh filename="package://pacsim/urdf/FL_Inside.stl" scale="0.01 0.01 0.01"/>
+        <mesh filename="package://pacsim/urdf/FL_Inside.stl" scale="0.01 0.01 0.01"/>
       </geometry>
-      </visual>
+    </visual>
   </link>
   <link name="FL_outside">
@@ -29,5 +29,5 @@
       <origin rpy="-1.57 0 0" xyz="0 0 0"/>
       <geometry>
-      <mesh filename="package://pacsim/urdf/FL_Outside.stl" scale="0.01 0.01 0.01"/>
+        <mesh filename="package://pacsim/urdf/FL_Outside.stl" scale="0.01 0.01 0.01"/>
       </geometry>
     </visual>
@@ -37,7 +37,7 @@
       <origin rpy="-1.57 0 0" xyz="0 0 0"/>
       <geometry>
-      <mesh filename="package://pacsim/urdf/FR_Inside.stl" scale="0.01 0.01 0.01"/>
+        <mesh filename="package://pacsim/urdf/FR_Inside.stl" scale="0.01 0.01 0.01"/>
       </geometry>
-      </visual>
+    </visual>
   </link>
   <link name="FR_outside">
@@ -45,5 +45,5 @@
       <origin rpy="-1.57 0 3.1415" xyz="0 0 0"/>
       <geometry>
-      <mesh filename="package://pacsim/urdf/FL_Outside.stl" scale="0.01 0.01 0.01"/>
+        <mesh filename="package://pacsim/urdf/FL_Outside.stl" scale="0.01 0.01 0.01"/>
       </geometry>
     </visual>
@@ -53,7 +53,7 @@
       <origin rpy="-1.57 0 0" xyz="0 0 0"/>
       <geometry>
-      <mesh filename="package://pacsim/urdf/RR_Inside.stl" scale="0.01 0.01 0.01"/>
+        <mesh filename="package://pacsim/urdf/RR_Inside.stl" scale="0.01 0.01 0.01"/>
       </geometry>
-      </visual>
+    </visual>
   </link>
   <link name="RR_outside">
@@ -61,5 +61,5 @@
       <origin rpy="-1.57 0 3.14" xyz="0 0 0"/>
       <geometry>
-      <mesh filename="package://pacsim/urdf/FL_Outside.stl" scale="0.01 0.01 0.01"/>
+        <mesh filename="package://pacsim/urdf/FL_Outside.stl" scale="0.01 0.01 0.01"/>
       </geometry>
     </visual>
@@ -69,7 +69,7 @@
       <origin rpy="-1.57 0 3.1415" xyz="0 0 0"/>
       <geometry>
-      <mesh filename="package://pacsim/urdf/RR_Inside.stl" scale="0.01 0.01 0.01"/>
+        <mesh filename="package://pacsim/urdf/RR_Inside.stl" scale="0.01 0.01 0.01"/>
       </geometry>
-      </visual>
+    </visual>
   </link>
   <link name="RL_outside">
@@ -77,5 +77,5 @@
       <origin rpy="-1.57 0 0" xyz="0 0 0"/>
       <geometry>
-      <mesh filename="package://pacsim/urdf/FL_Outside.stl" scale="0.01 0.01 0.01"/>
+        <mesh filename="package://pacsim/urdf/FL_Outside.stl" scale="0.01 0.01 0.01"/>
       </geometry>
     </visual>
@@ -85,5 +85,5 @@
       <origin rpy="0.0 0 0" xyz="0 0 0"/>
       <geometry>
-      <mesh filename="package://pacsim/urdf/Steering_Wheel.stl" scale="0.01 0.01 0.01"/>
+        <mesh filename="package://pacsim/urdf/Steering_Wheel.stl" scale="0.01 0.01 0.01"/>
       </geometry>
     </visual>

Commit message: hot-fix: back to old pacsim

File: src/pacsim/urdf/separate_model.xacro (robot description, xacro)
@@ -1,17 +1,17 @@
 <robot name="RosE" xmlns:xacro="http://www.ros.org/wiki/xacro">
   <xacro:property name="baseFrame" value="car" />
-  <link name="car">
+  <link name="${baseFrame}">
     <visual>
       <origin rpy="0.0 0 0" xyz="0 0 0"/>
-      <geometry>
+        <geometry>
         <cylinder radius="0.001" length=".001" />
       </geometry>
     </visual>
   </link>
-  <link name="Modell">
+   <link name="Modell">
     <visual>
-      <origin xyz="0 0 0" rpy="-1.57 0 0" />
+      <origin xyz="0 0 0" rpy="0 0 0" />
       <geometry>
-        <mesh filename="package://pacsim/urdf/Model_without_Steering_Tires.stl" scale="0.01 0.01 0.01"/>
+      <mesh filename="package://pacsim/urdf/Model_without_Steering_Tires.stl" scale="0.01 0.01 0.01"/>
       </geometry>
     </visual>
@@ -19,15 +19,15 @@
   <link name="FL_inside">
     <visual>
-      <origin rpy="-1.57 0 0" xyz="0 0 0"/>
+      <origin rpy="0.0 0 0" xyz="0 0 0"/>
       <geometry>
-        <mesh filename="package://pacsim/urdf/FL_Inside.stl" scale="0.01 0.01 0.01"/>
+      <mesh filename="package://pacsim/urdf/FL_Inside.stl" scale="0.01 0.01 0.01"/>
       </geometry>
-    </visual>
+      </visual>
   </link>
   <link name="FL_outside">
     <visual>
-      <origin rpy="-1.57 0 0" xyz="0 0 0"/>
+      <origin rpy="0.0 0 0" xyz="0 0 0"/>
       <geometry>
-        <mesh filename="package://pacsim/urdf/FL_Outside.stl" scale="0.01 0.01 0.01"/>
+      <mesh filename="package://pacsim/urdf/FL_Outside.stl" scale="0.01 0.01 0.01"/>
       </geometry>
     </visual>
@@ -35,15 +35,15 @@
   <link name="FR_inside">
     <visual>
-      <origin rpy="-1.57 0 0" xyz="0 0 0"/>
+      <origin rpy="0.0 0 0" xyz="0 0 0"/>
       <geometry>
-        <mesh filename="package://pacsim/urdf/FR_Inside.stl" scale="0.01 0.01 0.01"/>
+      <mesh filename="package://pacsim/urdf/FR_Inside.stl" scale="0.01 0.01 0.01"/>
       </geometry>
-    </visual>
+      </visual>
   </link>
   <link name="FR_outside">
     <visual>
-      <origin rpy="-1.57 0 3.1415" xyz="0 0 0"/>
+      <origin rpy="0.0 0 3.1415" xyz="0 0 0"/>
       <geometry>
-        <mesh filename="package://pacsim/urdf/FL_Outside.stl" scale="0.01 0.01 0.01"/>
+      <mesh filename="package://pacsim/urdf/FL_Outside.stl" scale="0.01 0.01 0.01"/>
       </geometry>
     </visual>
@@ -51,15 +51,15 @@
   <link name="RR_inside">
     <visual>
-      <origin rpy="-1.57 0 0" xyz="0 0 0"/>
+      <origin rpy="0.0 0 0" xyz="0 0 0"/>
       <geometry>
-        <mesh filename="package://pacsim/urdf/RR_Inside.stl" scale="0.01 0.01 0.01"/>
+      <mesh filename="package://pacsim/urdf/RR_Inside.stl" scale="0.01 0.01 0.01"/>
       </geometry>
-    </visual>
+      </visual>
   </link>
   <link name="RR_outside">
     <visual>
-      <origin rpy="-1.57 0 3.14" xyz="0 0 0"/>
+      <origin rpy="0.0 0 3.14" xyz="0 0 0"/>
       <geometry>
-        <mesh filename="package://pacsim/urdf/FL_Outside.stl" scale="0.01 0.01 0.01"/>
+      <mesh filename="package://pacsim/urdf/FL_Outside.stl" scale="0.01 0.01 0.01"/>
       </geometry>
     </visual>
@@ -67,15 +67,15 @@
   <link name="RL_inside">
     <visual>
-      <origin rpy="-1.57 0 3.1415" xyz="0 0 0"/>
+      <origin rpy="0.0 0 3.1415" xyz="0 0 0"/>
       <geometry>
-        <mesh filename="package://pacsim/urdf/RR_Inside.stl" scale="0.01 0.01 0.01"/>
+      <mesh filename="package://pacsim/urdf/RR_Inside.stl" scale="0.01 0.01 0.01"/>
       </geometry>
-    </visual>
+      </visual>
   </link>
   <link name="RL_outside">
     <visual>
-      <origin rpy="-1.57 0 0" xyz="0 0 0"/>
+      <origin rpy="0.0 0 0" xyz="0 0 0"/>
       <geometry>
-        <mesh filename="package://pacsim/urdf/FL_Outside.stl" scale="0.01 0.01 0.01"/>
+      <mesh filename="package://pacsim/urdf/FL_Outside.stl" scale="0.01 0.01 0.01"/>
       </geometry>
     </visual>
@@ -85,5 +85,5 @@
       <origin rpy="0.0 0 0" xyz="0 0 0"/>
       <geometry>
-        <mesh filename="package://pacsim/urdf/Steering_Wheel.stl" scale="0.01 0.01 0.01"/>
+      <mesh filename="package://pacsim/urdf/Steering_Wheel.stl" scale="0.01 0.01 0.01"/>
       </geometry>
     </visual>

Commit message: feat: back to pacsim functional

File: src/pacsim/urdf/separate_model.xacro (robot description, xacro)
@@ -1,17 +1,17 @@
 <robot name="RosE" xmlns:xacro="http://www.ros.org/wiki/xacro">
   <xacro:property name="baseFrame" value="car" />
-  <link name="${baseFrame}">
+  <link name="car">
     <visual>
       <origin rpy="0.0 0 0" xyz="0 0 0"/>
-        <geometry>
+      <geometry>
         <cylinder radius="0.001" length=".001" />
       </geometry>
     </visual>
   </link>
-   <link name="Modell">
+  <link name="Modell">
     <visual>
-      <origin xyz="0 0 0" rpy="0 0 0" />
+      <origin xyz="0 0 0" rpy="-1.57 0 0" />
       <geometry>
-      <mesh filename="package://pacsim/urdf/Model_without_Steering_Tires.stl" scale="0.01 0.01 0.01"/>
+        <mesh filename="package://pacsim/urdf/Model_without_Steering_Tires.stl" scale="0.01 0.01 0.01"/>
       </geometry>
     </visual>
@@ -19,15 +19,15 @@
   <link name="FL_inside">
     <visual>
-      <origin rpy="0.0 0 0" xyz="0 0 0"/>
+      <origin rpy="-1.57 0 0" xyz="0 0 0"/>
       <geometry>
-      <mesh filename="package://pacsim/urdf/FL_Inside.stl" scale="0.01 0.01 0.01"/>
+        <mesh filename="package://pacsim/urdf/FL_Inside.stl" scale="0.01 0.01 0.01"/>
       </geometry>
-      </visual>
+    </visual>
   </link>
   <link name="FL_outside">
     <visual>
-      <origin rpy="0.0 0 0" xyz="0 0 0"/>
+      <origin rpy="-1.57 0 0" xyz="0 0 0"/>
       <geometry>
-      <mesh filename="package://pacsim/urdf/FL_Outside.stl" scale="0.01 0.01 0.01"/>
+        <mesh filename="package://pacsim/urdf/FL_Outside.stl" scale="0.01 0.01 0.01"/>
       </geometry>
     </visual>
@@ -35,15 +35,15 @@
   <link name="FR_inside">
     <visual>
-      <origin rpy="0.0 0 0" xyz="0 0 0"/>
+      <origin rpy="-1.57 0 0" xyz="0 0 0"/>
       <geometry>
-      <mesh filename="package://pacsim/urdf/FR_Inside.stl" scale="0.01 0.01 0.01"/>
+        <mesh filename="package://pacsim/urdf/FR_Inside.stl" scale="0.01 0.01 0.01"/>
       </geometry>
-      </visual>
+    </visual>
   </link>
   <link name="FR_outside">
     <visual>
-      <origin rpy="0.0 0 3.1415" xyz="0 0 0"/>
+      <origin rpy="-1.57 0 3.1415" xyz="0 0 0"/>
       <geometry>
-      <mesh filename="package://pacsim/urdf/FL_Outside.stl" scale="0.01 0.01 0.01"/>
+        <mesh filename="package://pacsim/urdf/FL_Outside.stl" scale="0.01 0.01 0.01"/>
       </geometry>
     </visual>
@@ -51,15 +51,15 @@
   <link name="RR_inside">
     <visual>
-      <origin rpy="0.0 0 0" xyz="0 0 0"/>
+      <origin rpy="-1.57 0 0" xyz="0 0 0"/>
       <geometry>
-      <mesh filename="package://pacsim/urdf/RR_Inside.stl" scale="0.01 0.01 0.01"/>
+        <mesh filename="package://pacsim/urdf/RR_Inside.stl" scale="0.01 0.01 0.01"/>
       </geometry>
-      </visual>
+    </visual>
   </link>
   <link name="RR_outside">
     <visual>
-      <origin rpy="0.0 0 3.14" xyz="0 0 0"/>
+      <origin rpy="-1.57 0 3.14" xyz="0 0 0"/>
       <geometry>
-      <mesh filename="package://pacsim/urdf/FL_Outside.stl" scale="0.01 0.01 0.01"/>
+        <mesh filename="package://pacsim/urdf/FL_Outside.stl" scale="0.01 0.01 0.01"/>
       </geometry>
     </visual>
@@ -67,15 +67,15 @@
   <link name="RL_inside">
     <visual>
-      <origin rpy="0.0 0 3.1415" xyz="0 0 0"/>
+      <origin rpy="-1.57 0 3.1415" xyz="0 0 0"/>
       <geometry>
-      <mesh filename="package://pacsim/urdf/RR_Inside.stl" scale="0.01 0.01 0.01"/>
+        <mesh filename="package://pacsim/urdf/RR_Inside.stl" scale="0.01 0.01 0.01"/>
       </geometry>
-      </visual>
+    </visual>
   </link>
   <link name="RL_outside">
     <visual>
-      <origin rpy="0.0 0 0" xyz="0 0 0"/>
+      <origin rpy="-1.57 0 0" xyz="0 0 0"/>
       <geometry>
-      <mesh filename="package://pacsim/urdf/FL_Outside.stl" scale="0.01 0.01 0.01"/>
+        <mesh filename="package://pacsim/urdf/FL_Outside.stl" scale="0.01 0.01 0.01"/>
       </geometry>
     </visual>
@@ -85,5 +85,5 @@
       <origin rpy="0.0 0 0" xyz="0 0 0"/>
       <geometry>
-      <mesh filename="package://pacsim/urdf/Steering_Wheel.stl" scale="0.01 0.01 0.01"/>
+        <mesh filename="package://pacsim/urdf/Steering_Wheel.stl" scale="0.01 0.01 0.01"/>
       </geometry>
     </visual>
